File: LrTMAX.panel/LrTMAX_panel.kicad_pcb (KiCad board)
At the start: 2 copper layers, 0 parts

Commit message: Fix panels
Other:
- board text added: "12.75"
- board text added: "25"
- board text added: "37.5"
- board text added: "LrTMAX"
- board text removed: "30"
- board text removed: "40"
- board text removed: "LrE-6.8A"
Changed lines of the file:
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@@
   (general
     (thickness 1.6)
-    (drawings 118)
+    (drawings 111)
     (tracks 0)
     (zones 0)
@@
       (drillshape 0)
       (scaleselection 1)
-      (outputdirectory ""))
+      (outputdirectory "../LrTMAX.4lpb/Gerber/"))
   )
   (net 0 "")
@@
     (uvia_drill 0.1)
   )
-  (gr_line (start 135 132) (end 135 138) (layer Dwgs.User) (width 0.2))
-  (gr_line (start 125 132) (end 125 138) (layer Dwgs.User) (width 0.2))
-  (gr_line (start 115 132) (end 115 138) (layer Dwgs.User) (width 0.2))
-  (gr_line (start 105 132) (end 105 138) (layer Dwgs.User) (width 0.2))
-  (gr_line (start 95 132) (end 95 138) (layer Dwgs.User) (width 0.2))
-  (gr_line (start 85 132) (end 85 138) (layer Dwgs.User) (width 0.2))
-  (gr_line (start 75 132.2) (end 75 138.2) (layer Dwgs.User) (width 0.2))
-  (gr_line (start 65 132) (end 65 138) (layer Dwgs.User) (width 0.2))
+  (gr_line (start 135 134) (end 135 140) (layer Dwgs.User) (width 0.2))
+  (gr_line (start 125 134) (end 125 140) (layer Dwgs.User) (width 0.2))
+  (gr_line (start 115 134) (end 115 140) (layer Dwgs.User) (width 0.2))
+  (gr_line (start 105 134) (end 105 140) (layer Dwgs.User) (width 0.2))
+  (gr_line (start 95 134) (end 95 140) (layer Dwgs.User) (width 0.2))
+  (gr_line (start 85 134) (end 85 140) (layer Dwgs.User) (width 0.2))
+  (gr_line (start 75 134) (end 75 140) (layer Dwgs.User) (width 0.2))
+  (gr_line (start 65 134) (end 65 140) (layer Dwgs.User) (width 0.2))
   (gr_text 10 (at 129.9 158.3) (layer Dwgs.User)
     (effects (font (size 1.5 1.5) (thickness 0.3)))
@@
   (gr_line (start 115 155) (end 115 165) (layer Dwgs.User) (width 0.2))
   (gr_line (start 105 155) (end 105 165) (layer Dwgs.User) (width 0.2))
-  (gr_circle (center 130 120) (end 134 120) (layer Dwgs.User) (width 0.2))
-  (gr_line (start 65.2 120) (end 135.2 120) (layer Dwgs.User) (width 0.2))
-  (gr_line (start 70 115) (end 70 125) (layer Dwgs.User) (width 0.2))
-  (gr_line (start 90.2 114.9) (end 90.2 124.9) (layer Dwgs.User) (width 0.2))
-  (gr_circle (center 70 120) (end 74 120) (layer Dwgs.User) (width 0.2))
-  (gr_line (start 110 115) (end 110 125) (layer Dwgs.User) (width 0.2))
-  (gr_circle (center 110 120) (end 114 120) (layer Dwgs.User) (width 0.2))
-  (gr_line (start 130 115) (end 130 125) (layer Dwgs.User) (width 0.2))
-  (gr_circle (center 90 120) (end 94 120) (layer Dwgs.User) (width 0.2))
-  (gr_text LrE-6.8A (at 204.41412 173.609) (layer Dwgs.User)
+  (gr_circle (center 130 112.5) (end 134 112.5) (layer Dwgs.User) (width 0.2))
+  (gr_line (start 65.2 112.5) (end 135.2 112.5) (layer Dwgs.User) (width 0.2))
+  (gr_line (start 70 107.5) (end 70 117.5) (layer Dwgs.User) (width 0.2))
+  (gr_line (start 90 107.5) (end 90 117.5) (layer Dwgs.User) (width 0.2))
+  (gr_circle (center 70 112.5) (end 74 112.5) (layer Dwgs.User) (width 0.2))
+  (gr_line (start 110 107.5) (end 110 117.5) (layer Dwgs.User) (width 0.2))
+  (gr_circle (center 110 112.5) (end 114 112.5) (layer Dwgs.User) (width 0.2))
+  (gr_line (start 130 107.5) (end 130 117.5) (layer Dwgs.User) (width 0.2))
+  (gr_circle (center 90 112.5) (end 94 112.5) (layer Dwgs.User) (width 0.2))
+  (gr_text LrTMAX (at 204.41412 173.609) (layer Dwgs.User)
     (effects (font (size 3 3) (thickness 0.3)))
   )
@@
   (gr_line (start 135 155) (end 135 165) (layer Dwgs.User) (width 0.2))
   (gr_line (start 50 155) (end 50 165) (layer Dwgs.User) (width 0.2))
-  (gr_text 15 (at 157.1 143.4 90) (layer Dwgs.User)
-    (effects (font (size 1.5 1.5) (thickness 0.3)))
-  )
-  (gr_line (start 160 135) (end 160 150) (layer Dwgs.User) (width 0.2))
+  (gr_text 12.75 (at 157.1 143.4 90) (layer Dwgs.User)
+    (effects (font (size 1.5 1.5) (thickness 0.3)))
+  )
+  (gr_line (start 160 137.25) (end 160 150) (layer Dwgs.User) (width 0.2))
   (gr_line (start 155 150) (end 165 150) (layer Dwgs.User) (width 0.2))
   (gr_text 100 (at 27 101.1 90) (layer Dwgs.User)
@@
   (gr_line (start 50 30) (end 150 30) (layer Dwgs.User) (width 0.2))
   (gr_line (start 150 25) (end 150 45) (layer Dwgs.User) (width 0.2))
-  (gr_text 30 (at 35.6 105.6 90) (layer Dwgs.User)
+  (gr_text 25 (at 35.85 101.65 90) (layer Dwgs.User)
     (effects (font (size 1.5 1.5) (thickness 0.3)))
   )
@@
   )
   (gr_line (start 145 158.1) (end 150 158.1) (layer Dwgs.User) (width 0.2))
-  (gr_text 40 (at 35 73 90) (layer Dwgs.User)
+  (gr_text 37.5 (at 35 73 90) (layer Dwgs.User)
     (effects (font (size 1.5 1.5) (thickness 0.3)))
   )
@@
     (effects (font (size 1.5 1.5) (thickness 0.3)))
   )
-  (gr_line (start 37.5 97.5) (end 37.5 127.1) (layer Dwgs.User) (width 0.2))
+  (gr_line (start 37.5 50) (end 37.5 112.5) (layer Dwgs.User) (width 0.2))
   (gr_line (start 43.8 50) (end 43.8 54.9) (layer Dwgs.User) (width 0.2))
-  (gr_line (start 37.5 50) (end 37.5 97.5) (layer Dwgs.User) (width 0.2))
   (gr_line (start 150 155) (end 150 160) (layer Dwgs.User) (width 0.2))
   (gr_line (start 145 155) (end 145 160) (layer Dwgs.User) (width 0.2))
@@
   (gr_line (start 154 47.4) (end 145.2 54.6) (layer Dwgs.User) (width 0.2))
   (gr_line (start 162.5 47.4) (end 154 47.4) (layer Dwgs.User) (width 0.2))
-  (gr_line (start 155 135) (end 165 135) (layer Dwgs.User) (width 0.2))
-  (gr_line (start 45 120) (end 35 120) (layer Dwgs.User) (width 0.2))
-  (gr_line (start 35 90) (end 45 90) (layer Dwgs.User) (width 0.2))
+  (gr_line (start 155 137.25) (end 165 137.25) (layer Dwgs.User) (width 0.2))
+  (gr_line (start 45 112.5) (end 35 112.5) (layer Dwgs.User) (width 0.2))
+  (gr_line (start 35 87.5) (end 45 87.5) (layer Dwgs.User) (width 0.2))
   (gr_line (start 130 35.5) (end 130 45.5) (layer Dwgs.User) (width 0.2))
   (gr_line (start 110 35.5) (end 110 45.5) (layer Dwgs.User) (width 0.2))
@@
     (effects (font (size 1.5 1.5) (thickness 0.3)))
   )
-  (gr_line (start 151.3 120.9) (end 136.2 133.4) (layer Dwgs.User) (width 0.2))
+  (gr_line (start 151.3 120.9) (end 135.6 136.85) (layer Dwgs.User) (width 0.2))
   (gr_line (start 168.9 120.9) (end 151.3 120.9) (layer Dwgs.User) (width 0.2))
   (gr_text 8x8Φ (at 153.7 73.4) (layer Dwgs.User)
     (effects (font (size 1.5 1.5) (thickness 0.3)))
   )
-  (gr_line (start 144.4 75.4) (end 132.9 87) (layer Dwgs.User) (width 0.2))
+  (gr_line (start 144.4 75.4) (end 130.8 86.95) (layer Dwgs.User) (width 0.2))
   (gr_line (start 162.4 75.3) (end 144.5 75.3) (layer Dwgs.User) (width 0.2))
-  (gr_circle (center 135 135.05) (end 136.9 135.05) (layer Dwgs.User) (width 0.2))
-  (gr_circle (center 95 135) (end 96.9 135) (layer Dwgs.User) (width 0.2))
-  (gr_circle (center 125 135) (end 126.9 135) (layer Dwgs.User) (width 0.2))
-  (gr_circle (center 85 135) (end 86.9 135) (layer Dwgs.User) (width 0.2))
-  (gr_circle (center 115 135) (end 116.9 135) (layer Dwgs.User) (width 0.2))
-  (gr_circle (center 75 135) (end 76.9 135) (layer Dwgs.User) (width 0.2))
-  (gr_circle (center 105 135.1) (end 106.9 135.1) (layer Dwgs.User) (width 0.2))
-  (gr_circle (center 65 135) (end 66.9 135) (layer Dwgs.User) (width 0.2))
-  (gr_circle (center 130 90) (end 134 90) (layer Dwgs.User) (width 0.2))
-  (gr_circle (center 110 90) (end 114 90) (layer Dwgs.User) (width 0.2))
-  (gr_circle (center 90 90) (end 94 90) (layer Dwgs.User) (width 0.2))
-  (gr_circle (center 70 90) (end 74 90) (layer Dwgs.User) (width 0.2))
-  (gr_line (start 255.55 62.8) (end 255.55 92.8) (layer Dwgs.User) (width 0.2))
-  (gr_line (start 240.55 62.8) (end 240.55 92.8) (layer Dwgs.User) (width 0.2))
-  (gr_line (start 225.55 62.8) (end 225.55 92.8) (layer Dwgs.User) (width 0.2))
-  (gr_line (start 210.55 62.8) (end 210.55 92.8) (layer Dwgs.User) (width 0.2))
-  (gr_line (start 195.55 62.8) (end 195.55 92.8) (layer Dwgs.User) (width 0.2))
-  (gr_line (start 183.2 31.95) (end 258.2 31.95) (layer Dwgs.User) (width 0.2))
-  (gr_line (start 60 135) (end 140 135) (layer Dwgs.User) (width 0.2))
-  (gr_line (start 130.1 85) (end 130.1 95) (layer Dwgs.User) (width 0.2))
-  (gr_line (start 110 85) (end 110 95) (layer Dwgs.User) (width 0.2))
-  (gr_line (start 90 85) (end 90 95) (layer Dwgs.User) (width 0.2))
-  (gr_line (start 70 85) (end 70 95) (layer Dwgs.User) (width 0.2))
-  (gr_line (start 65 90) (end 135 90) (layer Dwgs.User) (width 0.2))
+  (gr_circle (center 135 137.25) (end 136.9 137.25) (layer Dwgs.User) (width 0.2))
+  (gr_circle (center 95 137.25) (end 96.9 137.25) (layer Dwgs.User) (width 0.2))
+  (gr_circle (center 125 137.25) (end 126.9 137.25) (layer Dwgs.User) (width 0.2))
+  (gr_circle (center 85 137.25) (end 86.9 137.25) (layer Dwgs.User) (width 0.2))
+  (gr_circle (center 115 137.25) (end 116.9 137.25) (layer Dwgs.User) (width 0.2))
+  (gr_circle (center 75 137.25) (end 76.9 137.25) (layer Dwgs.User) (width 0.2))
+  (gr_circle (center 105 137.25) (end 106.9 137.25) (layer Dwgs.User) (width 0.2))
+  (gr_circle (center 65 137.25) (end 66.9 137.25) (layer Dwgs.User) (width 0.2))
+  (gr_circle (center 130 87.5) (end 134 87.5) (layer Dwgs.User) (width 0.2))
+  (gr_circle (center 110 87.5) (end 114 87.5) (layer Dwgs.User) (width 0.2))
+  (gr_circle (center 90 87.5) (end 94 87.5) (layer Dwgs.User) (width 0.2))
+  (gr_circle (center 70 87.5) (end 74 87.5) (layer Dwgs.User) (width 0.2))
+  (gr_line (start 60 137.25) (end 140 137.25) (layer Dwgs.User) (width 0.2))
+  (gr_line (start 130 82.5) (end 130 92.5) (layer Dwgs.User) (width 0.2))
+  (gr_line (start 110 82.5) (end 110 92.5) (layer Dwgs.User) (width 0.2))
+  (gr_line (start 90 82.5) (end 90 92.5) (layer Dwgs.User) (width 0.2))
+  (gr_line (start 70 82.5) (end 70 92.5) (layer Dwgs.User) (width 0.2))
+  (gr_line (start 65 87.5) (end 135 87.5) (layer Dwgs.User) (width 0.2))
   (gr_circle (center 55 145) (end 56.6 145) (layer Dwgs.User) (width 0.2))
   (gr_circle (center 145 145) (end 146.6 145) (layer Dwgs.User) (width 0.2))
