File: LrTMAX.4lpb/LrTMAX.kicad_pcb (KiCad board)
At the start: 4 copper layers, 100 x 100 mm, 124 parts, among them J1 USB_B_Micro, J2 SM06B-SRSS-TB, Q1 2N7002, SW1 Tact_SW_8mm, SW10 EC11_SMD, SW11 EC11_SMD, SW12 EC11_SMD, SW13 EC11_SMD, SW14 EC11_SMD, SW15 EC11_SMD, SW16 EC11_SMD, SW17 EC11_SMD, SW2 Tact_SW_8mm, SW3 Tact_SW_8mm, SW4 Tact_SW_8mm, SW5 Tact_SW_8mm, SW6 Tact_SW_8mm, SW7 Tact_SW_8mm, SW8 Tact_SW_8mm, U1 STM32F072C8Tx, U3 SSD1306_OLED_0.91, U4 SPX3819M5-L3-3TR

Commit message: Fix panels
Routing:
- net GND: vias 16 -> 20
- net (no net): vias 0 -> 1

Commit message: Board fixes
Routing:
- net GND: track 64.1 -> 69.8 mm, vias 20 -> 45
- net /ENC2A: track 100.3 -> 102.5 mm
- net /ENC0A: track 91.7 -> 90.4 mm
- net /L2: track 107.8 -> 108.8 mm
- net (no net): vias 1 -> 0
